File: AntSniffer.kicad_pcb (KiCad board)
At the start: 4 copper layers, 50.1 x 30.1 mm, 6 parts, among them CN1 X2026WRS-2X09D-LPSW, CN2 X2026WRS-2X09D-LPSW, J1 Conn_01x10_MountingPin

Commit message: Add files via upload
Parts:
- CN1: footprint EASYEDA2KICAD:CONN-SMD_X2026WRS-2X09D-LPSW -> AntSniffer:CONN-TH_PHB-2-9AW; moved to B.Cu
- CN2: footprint EASYEDA2KICAD:CONN-SMD_X2026WRS-2X09D-LPSW -> AntSniffer:CN2-CONN-TH_PHB-2-9AW
- moved CN1 1.89 mm to (153.8, 57.8)
- moved CN2 1.87 mm to (183.3, 57.8), turned to -90 degrees
Connections:
- CN1 pad 11: /RX -> /TX
- CN1 pad 12: /TX -> /RX
- CN1 pad 15: /3V3 -> /RST
- CN1 pad 16: /RST -> /3V3
- CN1 pad 3: /SCL -> /SDA
- CN1 pad 4: /SDA -> /SCL
- CN1 pad 5: /A2 -> /PLUG
- CN1 pad 6: /PLUG -> /A2
- CN1 pad 7: /A0 -> /A1
- CN1 pad 8: /A1 -> /A0
- CN2 pad 1: unconnected-(CN2-Pad1) -> GND
- CN2 pad 11: /A0 -> /TX
- CN2 pad 12: /A1 -> /RX
- CN2 pad 13: /A2 -> GND
- CN2 pad 14: /PLUG -> GND
- CN2 pad 15: /SCL -> /RST
- CN2 pad 16: /SDA -> /3V3
- CN2 pad 17: GND -> unconnected-(CN1-Pad17)
- CN2 pad 18: GND -> unconnected-(CN1-Pad18)
- CN2 pad 2: unconnected-(CN2-Pad2) -> GND
- CN2 pad 3: /3V3 -> /SDA
- CN2 pad 4: /RST -> /SCL
- CN2 pad 5: GND -> /PLUG
- CN2 pad 6: GND -> /A2
- CN2 pad 7: /RX -> /A1
- CN2 pad 8: /TX -> /A0
Routing:
- net /TX: track 24.3 -> 28.4 mm
- net /RST: track 25.6 -> 29.7 mm
- net /PLUG: track 23.6 -> 27.7 mm
- net /A1: track 23.8 -> 27.9 mm
- net /SDA: track 24.0 -> 28.1 mm
- net GND: track 26.5 -> 26.0 mm, vias 12 -> 8
Other:
- board size 50.1 x 30.1 mm -> 48.6 x 30.1 mm
- board text removed: "Revision 1"
- board text removed: "The AntSniffer by OSMU"
